File: OV_Power/Motor_Driver.sch (KiCad schematic (older format))
At the start: 20 parts, among them CN1 CONN_HEADER_R_A_2POS_2.5MM, U3 LT6106, U4 VNH5019ATR-E

Commit message: Slight change to schemo per Rick's suggestion, also generated the real BOM.  Gerbers updated, should be ready for production.
Parts:
- R21: Mfr_PN (none) -> CSR2512A0R015F; Tolerance (none) -> 1%
Changed lines of the file:
@@
 F 9 "RES 0.015 OHM 1% 2W 2512" H 5500 1150 50  0001 C CNN "Desc"
 F 10 "15 mOhms ±1% 2W Chip Resistor 2512 (6432 Metric) Current Sense, Non-Inductive Metal Element" H 5500 1150 50  0001 C CNN "Detailed"
+F 11 "CSR2512A0R015F" H 5300 1150 50  0001 C CNN "Mfr_PN"
+F 12 "1%" H 5300 1150 50  0001 C CNN "Tolerance"
 	1    5300 1150
 	1    0    0    -1
