File: OV_Power/OV_Power.sch (KiCad schematic (older format))
At the start: 44 parts, among them J4 SpadeLug, J5 SpadeLug, Q1 SSM3K341R, Q2 2N7002BK, U1 LT3796, U2 LT1936

Commit message: Went through the Task list with Darren 1:1 with Ebony, possible new volunteer Changed gain on MPX4006DP to 8.5 gain Added a second MPXV4006GP Took sensor data off MCU: Pressure sensor (patient), oxygen sensor, flow sensor gain, flow sensor to be on FPGA only. Left alerts, battery sensor, and current measurements on MCU. Added circuit for Sensiron SM3020 and scaled output to 3v3.
Went through the Task list with Darren
1:1 with Ebony, possible new volunteer
Changed gain on MPX4006DP to 8.5 gain
Added a second MPXV4006GP
Took sensor data off MCU: Pressure sensor (patient), oxygen sensor, flow sensor gain, flow sensor to be on FPGA only. Left alerts, battery sensor, and current measurements on MCU.
Added circuit for Sensiron SM3020 and scaled output to 3v3.
Parts:
- C1, C14, C15, C4: symbol OpenVent:100nF_0603_Ceramic_Capacitor,_10%,_X7R,_25V -> OV_Power-rescue:100nF_0603_Ceramic_Capacitor,_10%,_X7R,_25V-OpenVent
- C2, C3: symbol OpenVent:10nF_0603_Ceramic_Capacitor,_10%,_50V,_X7R- -> OV_Power-rescue:10nF_0603_Ceramic_Capacitor,_10%,_50V,_X7R--OpenVent
- C5: symbol OpenVent:C_0603_0.22uf_25V_10% -> OV_Power-rescue:C_0603_0.22uf_25V_10%-OpenVent
- C6: symbol OpenVent:2.2uF_2824_film_capacitor_10%_40V -> OV_Power-rescue:2.2uF_2824_film_capacitor_10%_40V-OpenVent
- C7: symbol OpenVent:10uF_0805_Ceramic_Capacitor_10%_X7R_10V -> OV_Power-rescue:10uF_0805_Ceramic_Capacitor_10%_X7R_10V-OpenVent
- C8: symbol OpenVent:C_1210_10uF_25V_10%_X7R -> OV_Power-rescue:C_1210_10uF_25V_10%_X7R-OpenVent
- C9: symbol OpenVent:1uF_0603_Ceramic_Capacitor,_10%,_50V,_X5R -> OV_Power-rescue:1uF_0603_Ceramic_Capacitor,_10%,_50V,_X5R-OpenVent
- D1, D3: symbol OpenVent:MBRS260T3G -> OV_Power-rescue:MBRS260T3G-OpenVent
- D2: symbol OpenVent:MMBD914 -> OV_Power-rescue:MMBD914-OpenVent
- D4: symbol OpenVent:S1B -> OV_Power-rescue:S1B-OpenVent
- F1: symbol OpenVent:Polyfuse_10A -> OV_Power-rescue:Polyfuse_10A-OpenVent
- J4: symbol F_connectors:SpadeLug -> OV_Power-rescue:SpadeLug-F_connectors
- L1: symbol OV_Power-rescue:MSD1260-333-F_inductors -> OV_Power-rescue:MSD1260-333-F_inductors-OV_Power-rescue
- L2: symbol OpenVent:L_22uH_2.6A_42mOhm_SMT -> OV_Power-rescue:L_22uH_2.6A_42mOhm_SMT-OpenVent
- Q1: symbol OpenVent:SSM3K341R -> OV_Power-rescue:SSM3K341R-OpenVent
- Q2: symbol OpenVent:2N7002BK -> OV_Power-rescue:2N7002BK-OpenVent
- R1: symbol OpenVent:R_0603_806K_0.1W_1% -> OV_Power-rescue:R_0603_806K_0.1W_1%-OpenVent
- R10: symbol OpenVent:R_0805_050m_cursense -> OV_Power-rescue:R_0805_050m_cursense-OpenVent
- R11: symbol OpenVent:R_0603_015m_cursense -> OV_Power-rescue:R_0603_015m_cursense-OpenVent
- R12: symbol OpenVent:R_0603_53K_0.1W_1% -> OV_Power-rescue:R_0603_53K_0.1W_1%-OpenVent
- R13: symbol OpenVent:10k_0603_Chip_Resistor,_1%,_0.1W -> OV_Power-rescue:10k_0603_Chip_Resistor,_1%,_0.1W-OpenVent
- R14: symbol OpenVent:R_0603_49k9_0.1W_1% -> OV_Power-rescue:R_0603_49k9_0.1W_1%-OpenVent
- R15: symbol OpenVent:R_1206_250m_cursense -> OV_Power-rescue:R_1206_250m_cursense-OpenVent
- R16: symbol OpenVent:R_0603_113k_0.1W_1% -> OV_Power-rescue:R_0603_113k_0.1W_1%-OpenVent
- R17: symbol OpenVent:R_0603_30k1_0.1W_1% -> OV_Power-rescue:R_0603_30k1_0.1W_1%-OpenVent
- R18: symbol OpenVent:R_0603_95k3_0.1W_1% -> OV_Power-rescue:R_0603_95k3_0.1W_1%-OpenVent
- R19: symbol OpenVent:R_0603_10k2_0.1W_1% -> OV_Power-rescue:R_0603_10k2_0.1W_1%-OpenVent
- R2: symbol OpenVent:20k_0603_Chip_Resistor,_1%,_0.1W -> OV_Power-rescue:20k_0603_Chip_Resistor,_1%,_0.1W-OpenVent
- R3: symbol OpenVent:R_0603_499R_0.1W_1% -> OV_Power-rescue:R_0603_499R_0.1W_1%-OpenVent
- R4: symbol OpenVent:R_0603_40k2K_0.1W_1% -> OV_Power-rescue:R_0603_40k2K_0.1W_1%-OpenVent
- R5: symbol OpenVent:R_0603_19k6_0.1W_1% -> OV_Power-rescue:R_0603_19k6_0.1W_1%-OpenVent
- R6: symbol OpenVent:R_0603_499K_0.1W_1% -> OV_Power-rescue:R_0603_499K_0.1W_1%-OpenVent
- R7: symbol OpenVent:R_0603_97.6K_0.1W_1% -> OV_Power-rescue:R_0603_97.6K_0.1W_1%-OpenVent
- R8: symbol OpenVent:100K_0603_Chip_Resistor,_1%,_0.1W -> OV_Power-rescue:100K_0603_Chip_Resistor,_1%,_0.1W-OpenVent
- R9: symbol OpenVent:R_0603_2k_0.1W_1% -> OV_Power-rescue:R_0603_2k_0.1W_1%-OpenVent
- RT1: symbol OpenVent:R_Thermistor_0603_10K_NTC -> OV_Power-rescue:R_Thermistor_0603_10K_NTC-OpenVent
- U1: symbol F_ICs:LT3796 -> OV_Power-rescue:LT3796-F_ICs
- U2: symbol OpenVent:LT1936 -> OV_Power-rescue:LT1936-OpenVent
