File: LCD_FPGA.sch (KiCad schematic (older format))
At the start: 12 parts

Commit message: Created UI sheet, changed membrance switch lable to push button
Parts:
- removed C13, C2: 100nF_0603_Ceramic_Capacitor,_10%,_X7R,_25V, symbol OpenVent:100nF_0603_Ceramic_Capacitor,_10%,_X7R,_25V
- removed LCD1, LCD2: LCD_MOD_32DIG_16X2_TRANS_YLW_GRN, symbol OpenVent:LCD_MOD_32DIG_16X2_TRANS_YLW_GRN
- removed R34, R82: 3k6_0603_Chip_Resistor,_1%,_0.1W, symbol OpenVent:3k6_0603_Chip_Resistor,_1%,_0.1W
- removed R83, R84: 10k_0603_Chip_Resistor,_1%,_0.1W, symbol OpenVent:10k_0603_Chip_Resistor,_1%,_0.1W
- removed R? (x2): 100K_0603_Chip_Resistor,_1%,_0.1W, symbol OpenVent:100K_0603_Chip_Resistor,_1%,_0.1W
- removed U?: TXB0108, symbol OpenVent:TXB0108
- removed U?: TXB0104, symbol OpenVent:TXB0104
Connections:
- no-connect marks 2 -> 0
