File: AD_conv.sch (KiCad schematic (older format))
At the start: 30 parts, among them U9 74ACT244PW

Commit message: Revert "update ad_conv"
This reverts commit 2591c2734f3c7e5145f1228234b79b44e77147b9.
Parts:
- U9: value 74ACT244PW -> 74AHCT244
Changed lines of the file:
@@
 P 2650 2300
 F 0 "U9" H 2800 3100 50  0000 C CNN
-F 1 "74ACT244PW" H 2950 3000 50  0000 C CNN
+F 1 "74AHCT244" H 2950 3000 50  0000 C CNN
 F 2 "" H 2650 2300 50  0001 C CNN
 F 3 "https://assets.nexperia.com/documents/data-sheet/74AHC_AHCT244.pdf" H 2650 2300 50  0001 C CNN

Commit message: update ad_conv
Parts:
- U9: value 74AHCT244 -> 74ACT244PW
Changed lines of the file:
@@
 P 2650 2300
 F 0 "U9" H 2800 3100 50  0000 C CNN
-F 1 "74AHCT244" H 2950 3000 50  0000 C CNN
+F 1 "74ACT244PW" H 2950 3000 50  0000 C CNN
 F 2 "" H 2650 2300 50  0001 C CNN
 F 3 "https://assets.nexperia.com/documents/data-sheet/74AHC_AHCT244.pdf" H 2650 2300 50  0001 C CNN
