File: Speaker_Driver.sch (KiCad schematic (older format))
At the start: 0 parts

Commit message: Alarm Speaker Driver circuit added
Includes current measurement signals into FPGA
Parts:
- added C? (x10): 100nF_0603_Ceramic_Capacitor,_10%,_X7R,_25V, symbol OpenVent:100nF_0603_Ceramic_Capacitor,_10%,_X7R,_25V
- added C? (x2): 22uF_1206_Ceramic_Capacitor,_10%,_10V,_X7R, Resistor_SMD:R_1206_3216Metric, symbol OpenVent:22uF_1206_Ceramic_Capacitor,_10%,_10V,_X7R
- added C? (x2): 10nF_0603_Ceramic_Capacitor,_10%,_50V,_X7R-, symbol OpenVent:10nF_0603_Ceramic_Capacitor,_10%,_50V,_X7R-
- added C? (x2): 22nF_0603_Ceramic_Capacitor,_10%,_X7R,_50V, symbol OpenVent:22nF_0603_Ceramic_Capacitor,_10%,_X7R,_50V
- added L? (x4): SLF6028T-221MR26-PF, symbol OpenVent:SLF6028T-221MR26-PF
- added R? (x2): 1K_0603_Chip_Resistor,_1%,_0.1W, symbol OpenVent:1K_0603_Chip_Resistor,_1%,_0.1W
- added R? (x10): 10k_0603_Chip_Resistor,_1%,_0.1W, symbol OpenVent:10k_0603_Chip_Resistor,_1%,_0.1W
- added R? (x2): 12k_0603_Chip_Resistor,_1%,_0.1W, Resistor_SMD:R_0603_1608Metric, symbol OpenVent:12k_0603_Chip_Resistor,_1%,_0.1W
- added R? (x2): 62k_0603_Chip_Resistor,_1%,_0.1W, symbol OpenVent:62k_0603_Chip_Resistor,_1%,_0.1W
- added R? (x4): R_0603_3R0_0.1W_5%, symbol OpenVent:R_0603_3R0_0.1W_5%
- added R? (x2): 47k_0603_Chip_Resistor,_1%,_0.1W, symbol OpenVent:47k_0603_Chip_Resistor,_1%,_0.1W
- added R? (x2): R_0603_75K_0.1W_1%, symbol OpenVent:R_0603_75K_0.1W_1%
- added R? (x4): 100K_0603_Chip_Resistor,_1%,_0.1W, symbol OpenVent:100K_0603_Chip_Resistor,_1%,_0.1W
- added U? (x2): DRV8876, symbol OpenVent:DRV8876
Connections:
- new net: C?.1, R?.1, R?.2, U?.5 (VREF) (x2)
- new net: C?.1, C?.2 (x2)
- new net +3.3V: R?.1, R?.1, R?.1, R?.2
- new net +3V3: R?.1, R?.1, R?.1, R?.1, R?.1, R?.1
- new net +5V: C?.1, C?.1, C?.1, C?.1, C?.1, C?.1, U?.11 (VM), U?.11 (VM)
- new net GND: C?.2, C?.2, C?.2, C?.2, C?.2, C?.2, C?.2, C?.2, R?.1, R?.1, R?.1, R?.1, R?.1, R?.1, R?.2, R?.2, R?.2, R?.2, R?.2, R?.2, R?.2, R?.2, U?.15 (GND), U?.15 (GND), U?.17 (PAD), U?.17 (PAD), U?.9 (PGND), U?.9 (PGND)
- new net SPK1_CPH: C?.1, U?.13 (CPH)
- new net SPK1_CPL: C?.2, U?.14 (CPL)
- new net SPK1_EN: R?.2, U?.3 (nSLEEP)
- new net SPK1_FLT_N: R?.2, U?.4 (nFAULT)
- new net SPK1_FN: C?.2, L?.2, R?.1
- new net SPK1_FP: C?.1, L?.2, R?.1
- new net SPK1_IMODE: R?.2, U?.7 (IMODE)
- new net SPK1_IN1: U?.1 (EN_IN1)
- new net SPK1_IN1_REF: R?.1, R?.2
- new net SPK1_IN2: U?.2 (PH_IN2)
- new net SPK1_IN2_REF: R?.1, R?.1
- new net SPK1_N: R?.2
- new net SPK1_OUTN: L?.1, U?.10 (OUT2)
- new net SPK1_OUTP: L?.1, U?.8 (OUT1)
- new net SPK1_P: R?.2
- new net SPK1_PMODE: R?.2, R?.2, U?.16 (PMODE)
- new net SPK1_SENS: C?.1, R?.1, U?.6 (IPROPI)
- new net SPK1_VCP: C?.2, U?.12 (VCP)
- new net SPK2_CPH: C?.1, U?.13 (CPH)
- new net SPK2_CPL: C?.2, U?.14 (CPL)
- new net SPK2_EN: R?.2, U?.3 (nSLEEP)
- new net SPK2_FLT_N: R?.2, U?.4 (nFAULT)
- new net SPK2_FN: C?.2, L?.2, R?.1
- new net SPK2_FP: C?.1, L?.2, R?.1
- new net SPK2_IMODE: R?.2, U?.7 (IMODE)
- new net SPK2_IN1: U?.1 (EN_IN1)
- new net SPK2_IN1_REF: R?.1, R?.2
- new net SPK2_IN2: U?.2 (PH_IN2)
- new net SPK2_IN2_REF: R?.1, R?.2
- new net SPK2_N: R?.2
- new net SPK2_OUTN: L?.1, U?.10 (OUT2)
- new net SPK2_OUTP: L?.1, U?.8 (OUT1)
- new net SPK2_P: R?.2
- new net SPK2_PMODE: R?.2, R?.2, U?.16 (PMODE)
- new net SPK2_SENS: C?.1, R?.1, U?.6 (IPROPI)
- new net SPK2_VCP: C?.2, U?.12 (VCP)
Other:
- note added: "0"
- note added: "1"
- note added: "Brake, (Low-Side Slow Decay)"
- note added: "CURRENT COMPARISON"
- note added: "Coast, (H-Bridge Hi-Z)"
- note added: "DESCRIPTION"
- note added: "Do not fit"
- note added: "Forward (OUT1->OUT2)"
- note added: "H"
- note added: "Hi-Z"
- note added: "IN1"
- note added: "IN2"
- note added: "L"
- note added: "OUT1"
- note added: "OUT2"
- note added: "Reverse (OUT2->OUT1)"
- note added: "Sleep, (H-bridge Hi-Z)"
- note added: "TO EXTERNAL SPEAKER"
- note added: "Use local power and ground planes\nseparated from system planes,\nconnected at one point near power input"
- note added: "X"
- note added: "nSLEEP"
