File: Speaker_Driver.sch (KiCad schematic (older format))
At the start: 50 parts

Commit message: Rick's changes - April 19
Parts:
- removed R? (x2): 10k_0603_Chip_Resistor,_1%,_0.1W, symbol OpenVent:10k_0603_Chip_Resistor,_1%,_0.1W
- removed R?: 47k_0603_Chip_Resistor,_1%,_0.1W, symbol OpenVent:47k_0603_Chip_Resistor,_1%,_0.1W
- removed R?: R_0603_75K_0.1W_1%, symbol OpenVent:R_0603_75K_0.1W_1%
- removed R? (x2): 100K_0603_Chip_Resistor,_1%,_0.1W, symbol OpenVent:100K_0603_Chip_Resistor,_1%,_0.1W
- added R? (x2): 1K_0603_Chip_Resistor,_1%,_0.1W, symbol OpenVent:1K_0603_Chip_Resistor,_1%,_0.1W
Connections:
- net GND: now also R?.1, R?.1
- net SPK1_PMODE: now also R?.2
- net SPK2_PMODE: now also R?.2
- net 1.5V: now reaches C?.1, R?.1, R?.2, U?.5 (VREF)
- net SPK1_IN1_REF renamed SPK_HIGH_REF
- net SPK1_IN2_REF renamed SPK_LOW_REF
Other:
- note added: "1.05V"
- note added: "1.41V"
- note added: "TO EXTERNAL SPEAKER\nAdd Connector"
- note added: "Vsen = Iout * Rsens / 1000\n1.33V = 133 mA approx 0.8 W\n1.5V = 150 mA approx 1 W"
- note removed: "TO EXTERNAL SPEAKER"
- moved on the sheet: C?, L?, R?, U?
